File: gaia_obc.kicad_pcb (KiCad board)
At the start: 4 copper layers, 58 x 58 mm, 13 parts, among them J1 USB_C_Receptacle_USB2.0_16P, J2 Micro_SD_Card_Det2, J3 Conn_01x02_Pin, J6 Conn_01x10_Pin, J7 Conn_01x10_Pin, Q1 FS8205A, U1 CD-PA1616D, U2 LGS4056H, U3 DW01A, U4 USBLC6-2P6, U5 AP2112K-3.3, U6 ESP32-S3-PICO-1-N8R2, U7 WLR089U0-I_RM

Commit message: preparing ina3221
Parts:
- added J2: Micro_SD_Card_Det2, Connector_Card:microSD_HC_Hirose_DM3D-SF, F.Cu at (116.3, 31.6)
- added J3: Conn_01x02_Pin, Connector_Molex:Molex_MicroClasp_55935-0230_1x02_P2.00mm_Horizontal, F.Cu at (98.6, 71.6)
- added Q1: FS8205A, Package_TO_SOT_SMD:SOT-23-6, F.Cu at (94.4, 49.0)
- added U10: INA3221, Package_DFN_QFN:Texas_RGV0016A_VQFN-16-1EP_4x4mm_P0.65mm_EP2.1x2.1mm, F.Cu at (158.6, 105.7)
- added U2: LGS4056H, Package_DFN_QFN:DFN-8-1EP_3x3mm_P0.65mm_EP1.7x2.05mm, F.Cu at (110.1, 61.6)
- added U3: DW01A, Package_TO_SOT_SMD:SOT-23-6, F.Cu at (94.4, 53.7)
- added U5: AP2112K-3.3, Package_TO_SOT_SMD:SOT-23-5, F.Cu at (94.4, 58.3)
- added U7: WLR089U0-I_RM, OnionSAT_Gaia:MODULE_WLR089U0-I_RM, F.Cu at (100.4, 34.4)
- added U9: INA3221, Package_DFN_QFN:Texas_RGV0016A_VQFN-16-1EP_4x4mm_P0.65mm_EP2.1x2.1mm, F.Cu at (110.2, 49.8)
Other:
- board size 58 x 58 mm -> 50 x 52 mm

Commit message: creating psu switches
Parts:
- added J4: Conn_01x02_Pin, Connector_Molex:Molex_MicroClasp_55935-0230_1x02_P2.00mm_Horizontal, F.Cu at (152.9, 49.9)
- added U11: TPS22917DBV, Package_TO_SOT_SMD:SOT-23-6, F.Cu at (146.3, 53.8)
- added U12: TPS22917DBV, Package_TO_SOT_SMD:SOT-23-6, F.Cu at (146.3, 58.5)
- added U8: TPS22917DBV, Package_TO_SOT_SMD:SOT-23-6, F.Cu at (146.3, 49.2)
Connections:
- U5 pad 1: VCC -> Net-(U5-EN)
- U5 pad 3: VCC -> Net-(U5-EN)
- U9 pad 1: unconnected-(U9-IN-3-Pad1) -> VCC
- U9 pad 10: unconnected-(U9-PV-Pad10) -> Net-(U9-PV)
- U9 pad 11: unconnected-(U9-IN-1-Pad11) -> VCC
- U9 pad 12: unconnected-(U9-IN+1-Pad12) -> Net-(U9-IN+1)
- U9 pad 13: unconnected-(U9-TC-Pad13) -> Net-(U9-TC)
- U9 pad 14: unconnected-(U9-IN-2-Pad14) -> VCC
- U9 pad 15: unconnected-(U9-IN+2-Pad15) -> Net-(U9-IN+2)
- U9 pad 16: unconnected-(U9-VPU-Pad16) -> Net-(U9-VPU)
- U9 pad 17: unconnected-(U9-EP-Pad17) -> GND
- U9 pad 2: unconnected-(U9-IN+3-Pad2) -> Net-(U9-IN+3)
- U9 pad 3: unconnected-(U9-GND-Pad3) -> GND
- U9 pad 4: unconnected-(U9-VS-Pad4) -> +3.3V
- U9 pad 5: unconnected-(U9-A0-Pad5) -> +3.3V
- U9 pad 8: unconnected-(U9-WARNING-Pad8) -> Net-(U9-WARNING)
- U9 pad 9: unconnected-(U9-CRITICAL-Pad9) -> Net-(U9-CRITICAL)

Commit message: finishing psu
Parts:
- removed the J2 at (132.1, 99.7)
- removed the J2 at (116.3, 31.6)
- removed J3 (x2): Conn_01x02_Pin, Connector_Molex:Molex_MicroClasp_55935-0230_1x02_P2.00mm_Horizontal
- removed the Q1 at (94.4, 49.0)
- removed the Q1 at (159.6, 112.5)
- removed U2 (x2): LGS4056H, Package_DFN_QFN:DFN-8-1EP_3x3mm_P0.65mm_EP1.7x2.05mm
- removed the U3 at (94.4, 53.7)
- removed the U3 at (159.6, 117.2)
- removed the U5 at (94.4, 58.3)
- removed the U5 at (161.4, 121.6)
- removed the U7 at (100.4, 34.4)
- removed the U7 at (141.8, 98.4)
- added J2: Micro_SD_Card_Det2, Connector_Card:microSD_HC_Hirose_DM3D-SF, B.Cu at (225.9, 105.8)
- added Q1: FS8205A, Package_TO_SOT_SMD:SOT-23-6, F.Cu at (180.5, 114.4)
- added U13: INA3221, Package_DFN_QFN:Texas_RGV0016A_VQFN-16-1EP_4x4mm_P0.65mm_EP2.1x2.1mm, F.Cu at (218.5, 106.9)
- added U14: TPS22917DBV, Package_TO_SOT_SMD:SOT-23-6, F.Cu at (180.5, 99.0)
- added U15: TPS22917DBV, Package_TO_SOT_SMD:SOT-23-6, F.Cu at (185.1, 99.0)
- added U3: DW01A, Package_TO_SOT_SMD:SOT-23-6, F.Cu at (185.1, 114.4)
- added U5: AP2112K-3.3, Package_TO_SOT_SMD:SOT-23-5, F.Cu at (180.5, 109.3)
- added U7: WLR089U0-I_RM, OnionSAT_Gaia:MODULE_WLR089U0-I_RM, B.Cu at (227.0, 81.8)
- U10: value INA3221 -> TP4056-42-ESOP8; footprint Package_DFN_QFN:Texas_RGV0016A_VQFN-16-1EP_4x4mm_P0.65mm_EP2.1x2.1mm -> Package_SO:SOIC-8-1EP_3.9x4.9mm_P1.27mm_EP2.41x3.3mm_ThermalVias
- moved U1 170.5 mm to (226.8, 91.4)
- moved U9 138.2 mm to (235.8, 107.6)
- moved J1 92.6 mm to (225.9, 71.7)
- moved J6 80.3 mm to (210.2, 91.0), turned to 0 degrees
- moved U6 78.0 mm to (227.6, 103.9), turned to 90 degrees
- moved J7 72.9 mm to (242.8, 91.1), turned to 0 degrees
- moved U8 71.5 mm to (185.1, 109.3), turned to 90 degrees
- moved U4 71.4 mm to (218.7, 73.1), turned to 0 degrees
- moved U10 67.6 mm to (225.7, 113.5)
- moved U11 60.8 mm to (180.5, 104.1), turned to 90 degrees
- moved U12 59.9 mm to (185.1, 104.1), turned to 90 degrees
- moved J4 50.9 mm to (159.1, 100.3)
Connections:
- U10 pad 1: unconnected-(U10-IN-3-Pad1) -> GND
- U10 pad 2: unconnected-(U10-IN+3-Pad2) -> Net-(U10-PROG)
- U10 pad 3: unconnected-(U10-GND-Pad3) -> GND
- U10 pad 4: unconnected-(U10-VS-Pad4) -> VBUS
- U10 pad 5: unconnected-(U10-A0-Pad5) -> +BATT
- U10 pad 6: unconnected-(U10-SCL-Pad6) -> Net-(D2-K)
- U10 pad 7: unconnected-(U10-SDA-Pad7) -> Net-(D1-K)
- U10 pad 8: unconnected-(U10-WARNING-Pad8) -> VBUS
- U10 pad 9: unconnected-(U10-CRITICAL-Pad9) -> GND
- U9 pad 12: Net-(U9-IN+1) -> Net-(U8-VIN)
- U9 pad 15: Net-(U9-IN+2) -> Net-(U11-VIN)
- U9 pad 2: Net-(U9-IN+3) -> Net-(U12-VIN)
Routing:
- net GND: track 0.79 -> 0.00 mm
- removed copper zone on In2.Cu, net +3.3V
- removed copper zone on In1.Cu, net GND
Other:
- board size 50 x 52 mm -> 50 x 50 mm
- board text removed: "BOOT"
- board text removed: "On-Board Computer"
- board text removed: "WLR089 LoRa modul"

Commit message: Update gaia_obc.kicad_pcb
Parts:
- moved J6 162.2 mm to (48.1, 98.7)
- moved J2 162.2 mm to (65.5, 81.2), turned to 0 degrees
- moved U7 51.2 mm to (264.4, 46.9)
- moved J4 51.2 mm to (196.5, 65.4)
- moved J7 51.2 mm to (280.2, 56.1)
- moved U6 51.2 mm to (265.0, 68.9)
- moved U11 51.2 mm to (217.9, 69.1)
- moved U12 51.2 mm to (222.5, 69.1)
- moved J1 51.2 mm to (263.3, 36.7)
- moved Q1 51.2 mm to (217.9, 79.4)
- moved U1 51.2 mm to (264.2, 56.5)
- moved U10 51.2 mm to (263.1, 78.5)
- moved U13 51.2 mm to (255.9, 71.9)
- moved U14 51.2 mm to (217.9, 64.0)
- moved U15 51.2 mm to (222.5, 64.0)
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Other:
- outline, holes or cut-outs redrawn

Commit message: borad outline
Parts:
- removed J1: USB_C_Receptacle_USB2.0_16P, Connector_USB:USB_C_Receptacle_G-Switch_GT-USB-7010ASV
- removed J2: Micro_SD_Card_Det2, Connector_Card:microSD_HC_Hirose_DM3D-SF
- removed J4: Conn_01x02_Pin, Connector_Molex:Molex_MicroClasp_55935-0230_1x02_P2.00mm_Horizontal
- removed J6, J7: Conn_01x10_Pin, Connector_PinHeader_2.54mm:PinHeader_1x10_P2.54mm_Vertical_SMD_Pin1Left
- removed Q1: FS8205A, Package_TO_SOT_SMD:SOT-23-6
- removed U1: CD-PA1616D, OnionSAT_Gaia:XCVR_CD-PA1616D
- removed U10: TP4056-42-ESOP8, Package_SO:SOIC-8-1EP_3.9x4.9mm_P1.27mm_EP2.41x3.3mm_ThermalVias
- removed U11, U12, U14, U15, U8: TPS22917DBV, Package_TO_SOT_SMD:SOT-23-6
- removed U13, U9: INA3221, Package_DFN_QFN:Texas_RGV0016A_VQFN-16-1EP_4x4mm_P0.65mm_EP2.1x2.1mm
- removed U3: DW01A, Package_TO_SOT_SMD:SOT-23-6
- removed U4: USBLC6-2P6, Package_TO_SOT_SMD:SOT-666
- removed U5: AP2112K-3.3, Package_TO_SOT_SMD:SOT-23-5
- removed U6: ESP32-S3-PICO-1-N8R2, OnionSAT_Gaia:PQFN40P700X700X106-57N
- removed U7: WLR089U0-I_RM, OnionSAT_Gaia:MODULE_WLR089U0-I_RM
Other:
- outline, holes or cut-outs redrawn

Commit message: almost final release
Parts:
- added C1: 100nF, Capacitor_SMD:C_0402_1005Metric, F.Cu at (96.8, 86.1)
- added C10: 100nF, Capacitor_SMD:C_0402_1005Metric, F.Cu at (102.5, 88.1)
- added C11: 100nF, Capacitor_SMD:C_0402_1005Metric, F.Cu at (102.5, 90.0)
- added C12: 1uF, Capacitor_SMD:C_0402_1005Metric, F.Cu at (102.5, 92.0)
- added C13: 1uF, Capacitor_SMD:C_0402_1005Metric, F.Cu at (96.8, 74.2)
- added C14: 1uF, Capacitor_SMD:C_0402_1005Metric, F.Cu at (96.8, 76.2)
- added C15: 1uF, Capacitor_SMD:C_0402_1005Metric, F.Cu at (96.8, 78.2)
- added C16: 1uF, Capacitor_SMD:C_0402_1005Metric, F.Cu at (96.8, 80.2)
- added C17: 1uF, Capacitor_SMD:C_0402_1005Metric, F.Cu at (96.8, 82.1)
- added C2: 100nF, Capacitor_SMD:C_0402_1005Metric, F.Cu at (96.8, 88.1)
- added C23: 1uF, Capacitor_SMD:C_0402_1005Metric, F.Cu at (99.7, 74.2)
- added C24: 100nF, Capacitor_SMD:C_0402_1005Metric, F.Cu at (99.7, 76.2)
- added C25: 1uF, Capacitor_SMD:C_0402_1005Metric, F.Cu at (99.7, 78.2)
- added C26: 1uF, Capacitor_SMD:C_0402_1005Metric, F.Cu at (99.7, 80.2)
- added C27: 1uF, Capacitor_SMD:C_0402_1005Metric, F.Cu at (99.7, 82.1)
- added C28: 1uF, Capacitor_SMD:C_0402_1005Metric, F.Cu at (102.5, 74.2)
- added C29: 1uF, Capacitor_SMD:C_0402_1005Metric, F.Cu at (102.5, 76.2)
- added C3: 100nF, Capacitor_SMD:C_0402_1005Metric, F.Cu at (96.8, 90.0)
- added C30: 1uF, Capacitor_SMD:C_0402_1005Metric, F.Cu at (102.5, 78.2)
- added C31: 100nF, Capacitor_SMD:C_0402_1005Metric, F.Cu at (102.5, 80.2)
- added C32: 10uF, Capacitor_SMD:C_0402_1005Metric, F.Cu at (102.5, 82.1)
- added C33: 1uF, Capacitor_SMD:C_0402_1005Metric, F.Cu at (105.4, 74.2)
- added C34: 10uF, Capacitor_SMD:C_0402_1005Metric, F.Cu at (105.4, 76.2)
- added C35: 100nF, Capacitor_SMD:C_0402_1005Metric, F.Cu at (105.4, 78.2)
- added C36: 10uF, Capacitor_SMD:C_0402_1005Metric, F.Cu at (105.4, 80.2)
- added C37: 1uF, Capacitor_SMD:C_0402_1005Metric, F.Cu at (105.4, 82.1)
- added C38: 100nF, Capacitor_SMD:C_0402_1005Metric, F.Cu at (110.3, 74.2)
- added C39: 100nF, Capacitor_SMD:C_0402_1005Metric, F.Cu at (110.3, 76.2)
- added C4: 10uF, Capacitor_SMD:C_0402_1005Metric, F.Cu at (96.8, 92.0)
- added C40: 100nF, Capacitor_SMD:C_0402_1005Metric, F.Cu at (110.3, 78.2)
- added C41: 1uF, Capacitor_SMD:C_0402_1005Metric, F.Cu at (110.3, 80.2)
- added C42: 100nF, Capacitor_SMD:C_0402_1005Metric, F.Cu at (110.3, 82.1)
- added C5: 100nF, Capacitor_SMD:C_0402_1005Metric, F.Cu at (99.7, 86.1)
- added C6: 1uF, Capacitor_SMD:C_0402_1005Metric, F.Cu at (99.7, 88.1)
- added C7: 100nF, Capacitor_SMD:C_0402_1005Metric, F.Cu at (99.7, 90.0)
- added C8: 100nF, Capacitor_SMD:C_0402_1005Metric, F.Cu at (99.7, 92.0)
- added C9: 100nF, Capacitor_SMD:C_0402_1005Metric, F.Cu at (102.5, 86.1)
- added IC1: MAX17048G+T10, gaia_obc-footprints:SON50P200X200X80-9N-D, F.Cu at (-49.0, 125.8)
- added J1: USB_C_Receptacle_USB2.0_16P, Connector_USB:USB_C_Receptacle_G-Switch_GT-USB-7010ASV, F.Cu at (155.8, 74.9)
- added J2: Conn_02x10_Odd_Even, Connector_PinHeader_2.00mm:PinHeader_2x10_P2.00mm_Vertical_SMD, B.Cu at (185.1, 101.0)
- added J3: Conn_02x10_Odd_Even, Connector_PinHeader_2.00mm:PinHeader_2x10_P2.00mm_Vertical_SMD, B.Cu at (144.9, 101.5)
- added J4: Conn_01x02_Pin, Connector_Molex:Molex_MicroClasp_55935-0230_1x02_P2.00mm_Horizontal, F.Cu at (-63.9, 105.1)
- added J5: Micro_SD_Card_Det2, Connector_Card:microSD_HC_Hirose_DM3D-SF, F.Cu at (-33.6, 100.3)
- added J6: Conn_Coaxial_Small, Connector_Coaxial:SMA_Amphenol_132134-10_Vertical, F.Cu at (154.5, 86.2)
- added Q1: FS8205A, Package_TO_SOT_SMD:SOT-23-6, F.Cu at (-64.5, 94.5)
- added Q2: BSS138, Package_TO_SOT_SMD:SOT-23, F.Cu at (82.8, 115.8)
- added U1: ~, gaia_obc-footprints:kepernyo, F.Cu at (165.3, 103.0)
- added U1: USBLC6-2P6, Package_TO_SOT_SMD:SOT-666, F.Cu at (173.2, 122.0)
- added U10: TPS22917DBV, Package_TO_SOT_SMD:SOT-23-6, F.Cu at (-49.0, 99.1)
- added U11: AP2112K-3.3, Package_TO_SOT_SMD:SOT-23-5, F.Cu at (-59.4, 94.5)
- added U12: DW01A, Package_TO_SOT_SMD:SOT-23-6, F.Cu at (-80.4, 95.0)
- added U13: AP2112K-3.0, Package_TO_SOT_SMD:SOT-23-5, F.Cu at (105.4, 108.5)
- added U14: LGS4056HDB, Package_DFN_QFN:DFN-8-1EP_3x3mm_P0.65mm_EP1.55x2.4mm, F.Cu at (165.9, 120.1)
- added U15: CD-PA1616, gaia_obc-footprints:XCVR_CD-PA1616D, F.Cu at (91.0, 104.7)
- added U16: RFM95W-868S2, RF_Module:HOPERF_RFM9XW_SMD, F.Cu at (67.4, 63.6)
- added U2: MCP23017_ML, Package_DFN_QFN:QFN-28-1EP_6x6mm_P0.65mm_EP4.25x4.25mm, F.Cu at (100.7, 131.1)
- added U3: ESP32-S3-PICO-1-N8R2, gaia_obc-footprints:PQFN40P700X700X106-57N, B.Cu at (165.6, 95.3)
- added U4: INA3221, Package_DFN_QFN:Texas_RGV0016A_VQFN-16-1EP_4x4mm_P0.65mm_EP2.1x2.1mm, F.Cu at (-54.7, 105.2)
- added U5: INA3221, Package_DFN_QFN:Texas_RGV0016A_VQFN-16-1EP_4x4mm_P0.65mm_EP2.1x2.1mm, F.Cu at (-45.9, 85.5)
- added U6: TPS22917DBV, Package_TO_SOT_SMD:SOT-23-6, F.Cu at (-72.1, 102.5)
- added U7: TPS22917DBV, Package_TO_SOT_SMD:SOT-23-6, F.Cu at (-54.2, 94.5)
- added U8: TPS22917DBV, Package_TO_SOT_SMD:SOT-23-6, F.Cu at (-54.2, 99.1)
- added U9: TPS22917DBV, Package_TO_SOT_SMD:SOT-23-6, F.Cu at (-49.0, 94.5)

Commit message: prep for routing 2/1
Parts:
- added BZ1: Buzzer, gaia_obc-footprints:buzzer_MLT-5020, F.Cu at (177.0, 109.5)
- added C18: 1nF, Capacitor_SMD:C_0402_1005Metric, F.Cu at (143.3, 125.1)
- added C19: 1nF, Capacitor_SMD:C_0402_1005Metric, F.Cu at (143.3, 127.0)
- added C20: 1nF, Capacitor_SMD:C_0402_1005Metric, F.Cu at (143.3, 129.0)
- added C21: 1nF, Capacitor_SMD:C_0402_1005Metric, F.Cu at (143.3, 131.0)
- added C22: 1nF, Capacitor_SMD:C_0402_1005Metric, F.Cu at (143.3, 133.0)
- added D1: LED_Small, LED_SMD:LED_0603_1608Metric, F.Cu at (146.8, 125.4)
- added D2: LED_Small, LED_SMD:LED_0603_1608Metric, F.Cu at (146.8, 128.0)
- added D3: LED_Small, LED_SMD:LED_0603_1608Metric, F.Cu at (123.2, 158.5)
- added SW3: SW_Push, Button_Switch_SMD:SW_SPST_PTS647_Sx50, F.Cu at (135.5, 90.0)
- added SW4: SW_Push, Button_Switch_SMD:SW_SPST_PTS647_Sx50, F.Cu at (112.0, 133.0)
- added SW5: SW_Push, Button_Switch_SMD:SW_SPST_PTS647_Sx50, F.Cu at (112.6, 143.2)
- added SW6: SW_Push, Button_Switch_SMD:SW_SPST_PTS647_Sx50, F.Cu at (112.6, 151.8)
- added SW7: SW_Push, Button_Switch_SMD:SW_SPST_PTS647_Sx50, F.Cu at (150.0, 94.0)
- added U17: ~, gaia_obc-footprints:kepernyo, F.Cu at (130.5, 141.8)
- moved J1 9.30 mm to (165.0, 76.0), turned to 180 degrees

Commit message: almost routeable//98% done schema
Parts:
- removed C2: 100nF, Capacitor_SMD:C_0402_1005Metric
- removed C4: 10uF, Capacitor_SMD:C_0402_1005Metric
- removed the U1 at (165.3, 103.0)
- removed the U1 at (173.2, 122.0)
- added C43: 100nF, Capacitor_SMD:C_0402_1005Metric, F.Cu at (118.0, 44.3)
- added C44: 10uF, Capacitor_SMD:C_0402_1005Metric, F.Cu at (118.0, 46.3)
- added D10: LED_Small, LED_SMD:LED_0603_1608Metric, F.Cu at (108.8, 48.0)
- added D11: LED_Small, LED_SMD:LED_0603_1608Metric, F.Cu at (108.8, 50.5)
- added D12: LED_Small, LED_SMD:LED_0603_1608Metric, F.Cu at (108.8, 53.1)
- added D4: LED_Small, LED_SMD:LED_0603_1608Metric, F.Cu at (108.8, 32.4)
- added D5: LED_Small, LED_SMD:LED_0603_1608Metric, F.Cu at (108.8, 35.0)
- added D6: LED_Small, LED_SMD:LED_0603_1608Metric, F.Cu at (108.8, 37.6)
- added D7: LED_Small, LED_SMD:LED_0603_1608Metric, F.Cu at (108.8, 40.2)
- added D8: LED_Small, LED_SMD:LED_0603_1608Metric, F.Cu at (108.8, 42.8)
- added D9: LED_Small, LED_SMD:LED_0603_1608Metric, F.Cu at (108.8, 45.4)
- added R1: 10k, Resistor_SMD:R_0402_1005Metric, F.Cu at (86.6, 54.2)
- added R10: 10k, Resistor_SMD:R_0402_1005Metric, F.Cu at (89.5, 60.1)
- added R11: 10k, Resistor_SMD:R_0402_1005Metric, F.Cu at (89.5, 62.1)
- added R12: 10k, Resistor_SMD:R_0402_1005Metric, F.Cu at (89.5, 64.1)
- added R13: 10k, Resistor_SMD:R_0402_1005Metric, F.Cu at (92.4, 54.2)
- added R14: 10k, Resistor_SMD:R_0402_1005Metric, F.Cu at (104.7, 82.0)
- added R15: 10k, Resistor_SMD:R_0402_1005Metric, F.Cu at (104.7, 84.0)
- added R16: 10k, Resistor_SMD:R_0402_1005Metric, F.Cu at (104.7, 86.0)
- added R17: 10k, Resistor_SMD:R_0402_1005Metric, F.Cu at (104.7, 88.0)
- added R18: 10k, Resistor_SMD:R_0402_1005Metric, F.Cu at (104.7, 90.0)
- added R19: 10k, Resistor_SMD:R_0402_1005Metric, F.Cu at (107.6, 82.0)
- added R2: 10k, Resistor_SMD:R_0402_1005Metric, F.Cu at (86.6, 56.1)
- added R20: 10k, Resistor_SMD:R_0402_1005Metric, F.Cu at (107.6, 84.0)
- added R21: 10k, Resistor_SMD:R_0402_1005Metric, F.Cu at (107.6, 86.0)
- added R22: R_Small, Resistor_SMD:R_0603_1608Metric, F.Cu at (97.2, 82.3)
- added R23: R_Small, Resistor_SMD:R_0603_1608Metric, F.Cu at (97.2, 84.8)
- added R24: R_Small, Resistor_SMD:R_0603_1608Metric, F.Cu at (97.2, 87.3)
- added R25: R_Small, Resistor_SMD:R_0603_1608Metric, F.Cu at (97.2, 89.8)
- added R26: R_Small, Resistor_SMD:R_0603_1608Metric, F.Cu at (97.2, 92.3)
- added R27: R_Small, Resistor_SMD:R_0603_1608Metric, F.Cu at (97.2, 94.8)
- added R28: 0, Resistor_SMD:R_0402_1005Metric, F.Cu at (107.6, 88.0)
- added R29: 0, Resistor_SMD:R_0402_1005Metric, F.Cu at (107.6, 90.0)
- added R3: 10k, Resistor_SMD:R_0402_1005Metric, F.Cu at (86.6, 58.1)
- added R30: 0, Resistor_SMD:R_0402_1005Metric, F.Cu at (110.5, 82.0)
- added R31: 0, Resistor_SMD:R_0402_1005Metric, F.Cu at (110.5, 84.0)
- added R32: 0, Resistor_SMD:R_0402_1005Metric, F.Cu at (110.5, 86.0)
- added R33: 0, Resistor_SMD:R_0402_1005Metric, F.Cu at (110.5, 88.0)
- added R34: 0, Resistor_SMD:R_0402_1005Metric, F.Cu at (110.5, 90.0)
- added R35: 0, Resistor_SMD:R_0402_1005Metric, F.Cu at (113.4, 82.0)
- added R36: 0, Resistor_SMD:R_0402_1005Metric, F.Cu at (113.4, 84.0)
- added R37: 0, Resistor_SMD:R_0402_1005Metric, F.Cu at (113.4, 86.0)
- added R38: 100, Resistor_SMD:R_1206_3216Metric, F.Cu at (88.0, 96.5)
- added R39: TBA, Resistor_SMD:R_0402_1005Metric, F.Cu at (113.4, 88.0)
- added R4: 5.1k, Resistor_SMD:R_0402_1005Metric, F.Cu at (86.6, 60.1)
- added R40: TBA, Resistor_SMD:R_0402_1005Metric, F.Cu at (113.4, 90.0)
- added R41: 1k, Resistor_SMD:R_0603_1608Metric, F.Cu at (101.2, 82.3)
- added R42: 1, Resistor_SMD:R_0603_1608Metric, F.Cu at (101.2, 84.8)
- added R43: 1k, Resistor_SMD:R_0603_1608Metric, F.Cu at (101.2, 87.3)
- added R44: 100k, Resistor_SMD:R_0603_1608Metric, F.Cu at (101.2, 89.8)
- added R45: 100k, Resistor_SMD:R_0603_1608Metric, F.Cu at (101.2, 92.3)
- added R46: 470, Resistor_SMD:R_0402_1005Metric, F.Cu at (64.1, 76.4)
- added R47: 470, Resistor_SMD:R_0402_1005Metric, F.Cu at (64.1, 78.4)
- added R48: R_Small, Resistor_SMD:R_0402_1005Metric, F.Cu at (64.1, 80.4)
- added R49: 10k, Resistor_SMD:R_0402_1005Metric, F.Cu at (67.1, 76.4)
- added R5: 5.1k, Resistor_SMD:R_0402_1005Metric, F.Cu at (86.6, 62.1)
- added R50: 10, Resistor_SMD:R_0603_1608Metric, F.Cu at (73.9, 72.1)
- added R51: 10k, Resistor_SMD:R_0402_1005Metric, F.Cu at (67.1, 78.4)
- added R52: 10k, Resistor_SMD:R_0402_1005Metric, F.Cu at (67.1, 80.4)
- added R53: 10k, Resistor_SMD:R_0402_1005Metric, F.Cu at (70.0, 76.4)
- added R54: 10k, Resistor_SMD:R_0402_1005Metric, F.Cu at (70.0, 78.4)
- added R55: 10k, Resistor_SMD:R_0402_1005Metric, F.Cu at (70.0, 80.4)
- added R56: TBA, Resistor_SMD:R_0402_1005Metric, F.Cu at (92.4, 56.1)
- added R57: TBA, Resistor_SMD:R_0402_1005Metric, F.Cu at (92.4, 58.1)
- added R58: TBA, Resistor_SMD:R_0402_1005Metric, F.Cu at (92.4, 60.1)
- added R59: TBA, Resistor_SMD:R_0402_1005Metric, F.Cu at (92.4, 62.1)
- added R6: 10k, Resistor_SMD:R_0402_1005Metric, F.Cu at (86.6, 64.1)
- added R60: TBA, Resistor_SMD:R_0402_1005Metric, F.Cu at (92.4, 64.1)
- added R61: TBA, Resistor_SMD:R_0402_1005Metric, F.Cu at (95.3, 54.2)
- added R62: TBA, Resistor_SMD:R_0402_1005Metric, F.Cu at (95.3, 56.1)
- added R63: TBA, Resistor_SMD:R_0402_1005Metric, F.Cu at (95.3, 58.1)
- added R64: TBA, Resistor_SMD:R_0402_1005Metric, F.Cu at (95.3, 60.1)
- added R7: 10k, Resistor_SMD:R_0402_1005Metric, F.Cu at (89.5, 54.2)
- added R8: 10k, Resistor_SMD:R_0402_1005Metric, F.Cu at (89.5, 56.1)
- added R9: 10k, Resistor_SMD:R_0402_1005Metric, F.Cu at (89.5, 58.1)
- added U1: USBLC6-2P6, Package_TO_SOT_SMD:SOT-666, F.Cu at (98.8, 63.5)
- U3: moved to F.Cu
- moved U12 179.6 mm to (98.0, 74.2)
- moved U4 173.5 mm to (115.2, 70.3)
- moved U6 162.4 mm to (87.7, 74.2)
- moved U5 161.4 mm to (115.2, 76.6)
- moved U11 159.3 mm to (98.0, 69.6)
- moved J4 154.5 mm to (89.2, 84.1)
- moved Q1 154.3 mm to (87.7, 69.6)
- moved U8 150.0 mm to (92.9, 69.6)
- moved IC1 144.8 mm to (92.9, 97.0)
- moved U10 143.4 mm to (92.9, 78.8)
- moved U9 143.4 mm to (92.9, 74.2)
- moved U7 142.8 mm to (87.7, 78.8)
- moved D3 101.2 mm to (78.8, 67.5)
- moved U2 96.9 mm to (115.0, 35.2)
- moved J6 88.6 mm to (67.3, 70.8)
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Connections:
- C26 pad 2: /Power Supply Unit/VOUT_A1 -> /VOUT_A1
- C27 pad 2: /Power Supply Unit/VOUT_A2 -> /VOUT_A2
- C28 pad 2: /Power Supply Unit/VOUT_A3 -> /VOUT_A3
- C29 pad 2: /Power Supply Unit/VOUT_B1 -> /VOUT_B1
- C30 pad 2: /Power Supply Unit/VOUT_B2 -> /VOUT_B2
- J2 pad 10: unconnected-(J2-Pin_10-Pad10) -> SPI_0_SCLK
- J2 pad 11: unconnected-(J2-Pin_11-Pad11) -> /EXP2_USART_TXD
- J2 pad 12: unconnected-(J2-Pin_12-Pad12) -> /EXP0_USART_TXD
- J2 pad 13: unconnected-(J2-Pin_13-Pad13) -> /EXP2_USART_RXD
- J2 pad 14: unconnected-(J2-Pin_14-Pad14) -> /EXP0_USART_RXD
- J2 pad 17: unconnected-(J2-Pin_17-Pad17) -> GND
- J2 pad 18: unconnected-(J2-Pin_18-Pad18) -> GND
- J2 pad 19: unconnected-(J2-Pin_19-Pad19) -> GND
- J2 pad 20: unconnected-(J2-Pin_20-Pad20) -> GND
- J2 pad 5: unconnected-(J2-Pin_5-Pad5) -> /EXP1_SPI_CS
- J2 pad 6: unconnected-(J2-Pin_6-Pad6) -> SPI_0_MISO
- J2 pad 7: unconnected-(J2-Pin_7-Pad7) -> GND
- J2 pad 8: unconnected-(J2-Pin_8-Pad8) -> SPI_0_MOSI
- J2 pad 9: unconnected-(J2-Pin_9-Pad9) -> GND
- J3 pad 1: unconnected-(J3-Pin_1-Pad1) -> /VOUT_A1
- J3 pad 10: unconnected-(J3-Pin_10-Pad10) -> /VOUT_B2
- J3 pad 13: unconnected-(J3-Pin_13-Pad13) -> GND
- J3 pad 14: unconnected-(J3-Pin_14-Pad14) -> GND
- J3 pad 15: unconnected-(J3-Pin_15-Pad15) -> GND
- J3 pad 16: unconnected-(J3-Pin_16-Pad16) -> GND
- J3 pad 17: unconnected-(J3-Pin_17-Pad17) -> +BATT
- J3 pad 18: unconnected-(J3-Pin_18-Pad18) -> +BATT
- J3 pad 19: unconnected-(J3-Pin_19-Pad19) -> -BATT
- J3 pad 2: unconnected-(J3-Pin_2-Pad2) -> /VOUT_A1
- J3 pad 20: unconnected-(J3-Pin_20-Pad20) -> -BATT
- J3 pad 3: unconnected-(J3-Pin_3-Pad3) -> /VOUT_A2
- J3 pad 4: unconnected-(J3-Pin_4-Pad4) -> /VOUT_A2
- J3 pad 5: unconnected-(J3-Pin_5-Pad5) -> /VOUT_A3
- J3 pad 6: unconnected-(J3-Pin_6-Pad6) -> /VOUT_A3
- J3 pad 7: unconnected-(J3-Pin_7-Pad7) -> /VOUT_B1
- J3 pad 8: unconnected-(J3-Pin_8-Pad8) -> /VOUT_B1
- J3 pad 9: unconnected-(J3-Pin_9-Pad9) -> /VOUT_B2
- U10 pad 6: /Power Supply Unit/VOUT_B2 -> /VOUT_B2
- U2 pad 2: unconnected-(U2-GPB5-Pad2) -> Net-(D4-A)
- U2 pad 22: unconnected-(U2-GPA5-Pad22) -> Net-(D7-A)
- U2 pad 23: unconnected-(U2-GPA6-Pad23) -> Net-(D8-A)
- U2 pad 24: unconnected-(U2-GPA7-Pad24) -> Net-(D9-A)
- U2 pad 3: unconnected-(U2-GPB6-Pad3) -> Net-(D5-A)
- U2 pad 4: unconnected-(U2-GPB7-Pad4) -> Net-(D6-A)
- U3 pad 39: unconnected-(U3-GPIO34-Pad39) -> /EXP0_USART_TXD
- U3 pad 40: unconnected-(U3-GPIO35-Pad40) -> /EXP0_USART_RXD
- U3 pad 41: unconnected-(U3-GPIO36-Pad41) -> /EXP1_SPI_CS
- U3 pad 42: unconnected-(U3-GPIO37-Pad42) -> /EXP2_USART_TXD
- U3 pad 43: unconnected-(U3-GPIO38-Pad43) -> /EXP2_USART_RXD
- U3 pad 51: unconnected-(U3-GPIO45-Pad51) -> Net-(D11-A)
- U3 pad 52: unconnected-(U3-GPIO46-Pad52) -> Net-(D12-A)
- U6 pad 6: /Power Supply Unit/VOUT_A1 -> /VOUT_A1
- U7 pad 6: /Power Supply Unit/VOUT_A2 -> /VOUT_A2
- U8 pad 6: /Power Supply Unit/VOUT_A3 -> /VOUT_A3
- U9 pad 6: /Power Supply Unit/VOUT_B1 -> /VOUT_B1
Other:
- outline, holes or cut-outs redrawn
