File: gaia_obc.kicad_pcb (KiCad board)
At the start: 8 copper layers, 50 x 50 mm, 162 parts, among them IC1 MAX17048G+T10, J1 USB_C_Receptacle_USB2.0_16P, J2 Conn_02x10_Odd_Even, J3 Conn_02x10_Odd_Even, J5 Micro_SD_Card_Det2, J6 Conn_Coaxial_Small, Q1 IRLML6244, Q2 FS8205A, Q3 BSS138, SW1 SW_Push, SW2 SW_Push, SW3 SW_Push, SW4 SW_Push, SW5 SW_Push, SW6 SW_Push, SW7 SW_Push, SW8 SW_Slide_DPDT, U1 MCP23017_ML, U10 TPS22917DBV, U11 AP2112K-3.3, U12 DW01A, U13 AP2112K-3.0, U14 LGS4056HDB, U15 CD-PA1616, U16 RFM95W-868S2, U17 BME280, U2 USBLC6-2P6, U3 ESP32-S3-PICO-1-N8R2, U4 INA3221, U5 INA3221, U6 TPS22917DBV, U7 TPS22917DBV, U8 TPS22917DBV, U9 TPS22917DBV

Commit message: finalizing everything + creating stencil + ORDER 08. 25.
Parts:
- J6: footprint Connector_Coaxial:SMA_Amphenol_132134_Vertical -> gaia_obc-footprints:SMA-TH_HL-SMA-KHD2
Other:
- board text added: "On-Board Computer"
- board text added: "revision 1.0 Designed by Tamás Pécsi"
