File: gaia_obc.kicad_pcb (KiCad board)
At the start: 8 copper layers, 50 x 50 mm, 162 parts, among them IC1 MAX17048G+T10, J1 USB_C_Receptacle_USB2.0_16P, J2 Conn_02x10_Odd_Even, J3 Conn_02x10_Odd_Even, J5 Micro_SD_Card_Det2, J6 Conn_Coaxial_Small, Q1 IRLML6244, Q2 FS8205A, Q3 BSS138, SW1 SW_Push, SW2 SW_Push, SW3 SW_Push, SW4 SW_Push, SW5 SW_Push, SW6 SW_Push, SW7 SW_Push, SW8 SW_Slide_DPDT, U1 MCP23017_ML, U10 TPS22917DBV, U11 AP2112K-3.3, U12 DW01A, U13 AP2112K-3.0, U14 LGS4056HDB, U15 CD-PA1616, U16 RFM95W-868S2, U17 BME280, U2 USBLC6-2P6, U3 ESP32-S3-PICO-1-N8R2, U4 INA3221, U5 INA3221, U6 TPS22917DBV, U7 TPS22917DBV, U8 TPS22917DBV, U9 TPS22917DBV

Commit message: obc v1.2-pre1
Parts:
- removed D1: LED_Small, LED_SMD:LED_0603_1608Metric
- removed R43, R44, R45, R46, R47: 0, Resistor_SMD:R_0402_1005Metric
- removed R6: TBA, Resistor_SMD:R_0402_1005Metric
- D10, D11: footprint LED_SMD:LED_0603_1608Metric -> LED_SMD:LED_0805_2012Metric
- moved D11 36.0 mm to (175.8, 123.8), turned to 90 degrees
- moved D10 34.8 mm to (173.7, 123.8), turned to 90 degrees
- moved R50 32.5 mm to (175.8, 121.1), turned to -90 degrees
- moved R49 31.2 mm to (173.7, 121.1), turned to 90 degrees
- moved R7 6.29 mm to (144.3, 112.2)
- moved D2 6.29 mm to (141.7, 112.2)
- moved R8 5.51 mm to (144.3, 109.3)
- moved D3 5.50 mm to (141.7, 109.3)
- moved R9 4.72 mm to (144.3, 106.5)
- moved D4 4.72 mm to (141.8, 106.5)
- moved R10 3.94 mm to (144.3, 103.6)
- moved D5 3.93 mm to (141.8, 103.6)
- moved R11 3.15 mm to (144.3, 100.7)
- moved D6 3.14 mm to (141.8, 100.7)
- moved R12 2.37 mm to (144.3, 97.8)
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Connections:
- R49 pad 1: Net-(D10-K) -> Net-(D10-A)
- R50 pad 2: Net-(D11-K) -> Net-(D11-A)
- U14 pad 6: Net-(D11-A) -> Net-(D11-K)
- U14 pad 7: Net-(D10-A) -> Net-(D10-K)
Routing:
- net Net-(D11-A): track 40.4 -> 1.20 mm, vias 2 -> 0
- net Net-(D10-A): track 38.9 -> 1.21 mm, vias 2 -> 0
- net VBUS: track 78.1 -> 43.1 mm, vias 2 -> 1
- net Net-(D10-K): track 1.51 -> 12.4 mm, vias 0 -> 2
- net GND: track 132.3 -> 142.8 mm, vias 223 -> 222
- net Net-(D11-K): track 1.50 -> 11.2 mm, vias 0 -> 2
- net /SCREEN_MOSI: track 27.4 -> 35.9 mm
- net +3V0: track 28.9 -> 37.0 mm, vias 2 -> 4
- net Net-(D3-A): track 22.2 -> 16.2 mm
- net /SCREEN_CLK: track 33.4 -> 39.4 mm
- net Net-(D4-A): track 26.3 -> 21.5 mm
- net Net-(U18-LEDK): track 17.1 -> 21.7 mm
- net /SCREEN_DC: track 26.2 -> 30.4 mm
- net Net-(D5-A): track 20.6 -> 17.4 mm
- net Net-(D2-A): track 21.7 -> 18.7 mm
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Other:
- board text added: "BOOT"
- board text added: "CHRG"
- board text added: "GPS FIX"
- board text added: "LORA ANT"
- board text added: "LORA RX"
- board text added: "LORA TX"
- board text added: "PCYC"
- board text added: "PWR A1"
- board text added: "PWR A2"
- board text added: "PWR A3"
- board text added: "PWR B1"
- board text added: "PWR B2"
- board text added: "STBY"
- board text added: "SYSTEM"
- board text added: "revision 1.2 Designed by Tamás Pécsi"
- board text removed: "revision 1.1 Designed by Tamás Pécsi"

Commit message: v1.2
Parts:
- removed C33: 10uF, Capacitor_SMD:C_0603_1608Metric
- removed IC1: MAX17048G+T10, gaia_obc-footprints:SON50P200X200X80-9N-D
- removed R54, R55: 100k, Resistor_SMD:R_0603_1608Metric
- added C49: 1uF, Capacitor_SMD:C_0603_1608Metric, F.Cu at (185.2, 101.5)
- added R6: 0.01R, Resistor_SMD:R_2512_6332Metric, F.Cu at (187.7, 107.6)
- added U19: INA238/INA237, gaia_obc-footprints:VSSOP-10_3x3mm_P0.5mm, F.Cu at (187.6, 100.2)
Connections:
- J3 pad 17: +BATT -> PRI_HI
- J3 pad 18: +BATT -> PRI_HI
Routing:
- net I2C_1_SCL: track 116.6 -> 145.4 mm, vias 11 -> 12
- net I2C_1_SDA: track 132.4 -> 156.9 mm
- net PRI_HI: track 0.00 -> 12.2 mm, vias 0 -> 1
- net +3.3V: track 78.9 -> 85.5 mm, vias 32 -> 33
- net Net-(IC1-~{ALRT}): track 6.31 -> 0.00 mm, vias 2 -> 0
- net Net-(IC1-QSTRT): track 4.95 -> 0.00 mm, vias 2 -> 0
- net +BATT: track 38.3 -> 34.5 mm, vias 4 -> 2
- net Net-(D2-K): track 0.00 -> 1.30 mm
- net Net-(D12-K): track 0.00 -> 1.22 mm
- net Net-(D9-A): track 14.7 -> 13.5 mm
- net /USB_D-: track 36.4 -> 35.4 mm
- net GND: track 142.8 -> 143.1 mm, vias 222 -> 230
Other:
- board text added: "OFF"
- board text added: "ON"
- board text added: "revision 1.2 Designed by T. Pécsi"
- board text removed: "revision 1.2 Designed by Tamás Pécsi"

Commit message: Update gaia_obc.kicad_pcb
Routing:
- net VBUS: track 43.1 -> 40.3 mm
- net -BATT: track 11.2 -> 9.72 mm
Changed lines of the file:
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@@
 	)
 	(gr_rect
-		(start 153.36917 119.826325)
-		(end 153.1 120.026351)
+		(start 153.1 119.826325)
+		(end 153.36917 120.026351)
 		(stroke
 			(width 0.14)
@@
 	)
 	(gr_rect
-		(start 162.059147 119.826327)
-		(end 160.733054 120.085618)
+		(start 160.733054 119.826327)
+		(end 162.059147 120.085618)
 		(stroke
 			(width 0.14)
@@
 	)
 	(gr_rect
-		(start 153.3667 120.339971)
-		(end 153.1 121.55)
+		(start 153.1 120.339971)
+		(end 153.3667 121.55)
 		(stroke
 			(width 0.14)
@@
 	)
 	(gr_rect
-		(start 161.530685 120.39183)
-		(end 161.266454 121.55)
+		(start 161.266454 120.39183)
+		(end 161.530685 121.55)
 		(stroke
 			(width 0.14)
@@
 	)
 	(segment
+		(start 174.816 116.784)
+		(end 174.6 117)
+		(width 0.35)
+		(layer "B.Cu")
+		(net 1)
+	)
+	(segment
 		(start 169.8 118.547658)
 		(end 169.8 117.8955)
@@
 	)
 	(segment
-		(start 174.366994 119.41498)
-		(end 174.366994 118.709954)
-		(width 0.35)
-		(layer "B.Cu")
-		(net 1)
-	)
-	(segment
 		(start 181.029694 112.444)
 		(end 181.296 112.710306)
@@
 	)
 	(segment
-		(start 176.056 119.171986)
-		(end 175.38948 119.838506)
-		(width 0.35)
-		(layer "B.Cu")
-		(net 1)
-	)
-	(segment
 		(start 169.8 117.8955)
 		(end 169.8 117.2435)
@@
 	(segment
 		(start 176.056 116.784)
-		(end 176.056 119.171986)
+		(end 174.816 116.784)
 		(width 0.35)
 		(layer "B.Cu")
@@
 	)
 	(segment
+		(start 174.6 117)
+		(end 174.6 117.8955)
+		(width 0.35)
+		(layer "B.Cu")
+		(net 1)
+	)
+	(segment
 		(start 174.366994 118.709954)
 		(end 174.6 118.476948)
@@
 	)
 	(segment
-		(start 175.38948 119.838506)
-		(end 174.79052 119.838506)
-		(width 0.35)
-		(layer "B.Cu")
-		(net 1)
-	)
-	(segment
 		(start 170.61 119.35)
 		(end 170.602342 119.35)
@@
 	)
 	(segment
-		(start 174.79052 119.838506)
-		(end 174.366994 119.41498)
-		(width 0.35)
-		(layer "B.Cu")
-		(net 1)
-	)
-	(segment
 		(start 174.6 118.476948)
 		(end 174.6 117.8955)
@@
 	)
 	(segment
-		(start 187.35 112.2)
-		(end 187.675 112.525)
-		(width 0.6)
-		(layer "B.Cu")
-		(net 15)
-	)
-	(segment
-		(start 186.099999 112.2)
-		(end 187.35 112.2)
+		(start 187.675 110.091938)
+		(end 187.28 109.696938)
 		(width 0.6)
 		(layer "B.Cu")
@@
 	)
 	(segment
-		(start 187.675 112.525)
-		(end 187.675 113.4)
+		(start 187.675 113.4)
+		(end 186.3625 113.4)
 		(width 0.6)
 		(layer "B.Cu")
@@
 	)
 	(segment
-		(start 186.099999 110.876939)
-		(end 187.28 109.696938)
-		(width 0.6)
-		(layer "B.Cu")
-		(net 15)
-	)
-	(segment
-		(start 186.099999 112.2)
-		(end 186.099999 110.876939)
+		(start 187.675 113.4)
+		(end 187.675 110.091938)
 		(width 0.6)
 		(layer "B.Cu")
@@
 	)
 	(segment
-		(start 186.099999 113.6625)
-		(end 186.099999 112.2)
+		(start 186.3625 113.4)
+		(end 186.1 113.6625)
 		(width 0.6)
 		(layer "B.Cu")

Commit message: adding logos + generating production files
Parts:
- J5: footprint Connector_Card:microSD_HC_Hirose_DM3D-SF -> gaia_obc-footprints:microSD_HC_Hirose_DM3D-SF
Routing:
- net +3.3V: track 85.5 -> 86.1 mm
Other:
- board text added: "A. B-Sörös M. Dernovics R. Mihályffy Z. Mihályffy D. Nagy T. Pécsi"
- board text added: "CPWR"
- board text added: "Follow us on Social Media"
- board text added: "designed for CanSat 2026"
- board text added: "revision 1.2 Project Neptune"
- board text removed: "PCYC"
- board text removed: "revision 1.2 Designed by T. Pécsi"
