File: gaia_obc_dmu.kicad_sch (KiCad schematic)
At the start: 29 parts, among them J5 Micro_SD_Card_Det2, J6 Conn_Coaxial_Small, Q3 BSS138, SW3 SW_Push, SW4 SW_Push, SW5 SW_Push, SW6 SW_Push, SW7 SW_Push, U15 CD-PA1616, U16 RFM95W-868S2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

Commit message: finalizing everything + creating stencil + ORDER 08. 25.
Parts:
- J6: footprint Connector_Coaxial:SMA_Amphenol_132134_Vertical -> gaia_obc-footprints:SMA-TH_HL-SMA-KHD2
- Q3: footprint Package_TO_SOT_SMD:SOT-23 -> gaia_obc-footprints:SOT-23
- U16: footprint RF_Module:HOPERF_RFM9XW_SMD -> gaia_obc-footprints:HOPERF_RFM9XW_SMD
- U17: footprint Package_LGA:Bosch_LGA-8_2.5x2.5mm_P0.65mm_ClockwisePinNumbering -> gaia_obc-footprints:Bosch_LGA-8_2.5x2.5mm_P0.65mm_ClockwisePinNumbering
Changed lines of the file:
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@@
 			)
 		)
-		(property "Footprint" "RF_Module:HOPERF_RFM9XW_SMD"
+		(property "Footprint" "gaia_obc-footprints:HOPERF_RFM9XW_SMD"
 			(at -12.7 119.38 0)
 			(effects
@@
 		(dnp no)
 		(property "Reference" "C40"
-			(at 101.346 45.466 0)
+			(at 102.616 45.466 0)
 			(effects
 				(font
@@
 			)
 		)
-		(property "Footprint" "Package_LGA:Bosch_LGA-8_2.5x2.5mm_P0.65mm_ClockwisePinNumbering"
+		(property "Footprint" "gaia_obc-footprints:Bosch_LGA-8_2.5x2.5mm_P0.65mm_ClockwisePinNumbering"
 			(at 190.5 151.13 0)
 			(effects
@@
 			)
 		)
-		(property "Footprint" "Connector_Coaxial:SMA_Amphenol_132134_Vertical"
+		(property "Footprint" "gaia_obc-footprints:SMA-TH_HL-SMA-KHD2"
 			(at 104.14 153.67 0)
 			(effects
@@
 			)
 		)
-		(property "Footprint" "Package_TO_SOT_SMD:SOT-23"
+		(property "Footprint" "gaia_obc-footprints:SOT-23"
 			(at 165.1 74.295 0)
 			(effects

Commit message: Cleaning up schematics
Parts:
- R58: value R_Small -> TBA
Other:
- title: (none) -> GAIA On-Board Computer
