File: gaia_obc_dmu.kicad_sch (KiCad schematic)
At the start: 29 parts, among them J5 Micro_SD_Card_Det2, J6 Conn_Coaxial_Small, Q3 BSS138, SW3 SW_Push, SW4 SW_Push, SW5 SW_Push, SW6 SW_Push, SW7 SW_Push, U15 CD-PA1616, U16 RFM95W-868S2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

Commit message: v1.3
Connections:
- net VBACKUP: now reaches U15.4 (VBACKUP)
- no-connect marks 16 -> 15
Changed lines of the file:
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@@
 	)
 	(no_connect
-		(at 86.36 91.44)
-	)
-	(no_connect
 		(at 36.83 33.02)
 	)
@@
 	(wire
 		(pts
+			(xy 90.17 91.44) (xy 86.36 91.44)
+		)
+		(stroke
+			(width 0)
+			(type default)
+		)
+	)
+	(wire
+		(pts
 			(xy 96.52 86.36) (xy 96.52 88.9)
 		)
@@
 					(unit 1)
 				)
+			)
+		)
+	)
+	(symbol
+		(lib_id "power:VDC")
+		(at 90.17 91.44 270)
+		(unit 1)
+		(exclude_from_sim no)
+		(in_bom yes)
+		(on_board yes)
+		(dnp no)
+		(fields_autoplaced yes)
+		(property "Reference" "#PWR0193"
+			(at 86.36 91.44 0)
+			(effects
+				(font
+					(size 1.27 1.27)
+				)
+				(hide yes)
+			)
+		)
+		(property "Value" "VBACKUP"
+			(at 93.98 91.4399 90)
+			(effects
+				(font
+					(size 1.27 1.27)
+				)
+				(justify left)
+			)
+		)
+		(property "Footprint" ""
+			(at 90.17 91.44 0)
+			(effects
+				(font
+					(size 1.27 1.27)
+				)
+				(hide yes)
+			)
+		)
+		(property "Datasheet" ""
+			(at 90.17 91.44 0)
+			(effects
+				(font
+					(size 1.27 1.27)
+				)
+				(hide yes)
+			)
+		)
+		(property "Description" "Power symbol creates a global label with name \"VDC\""
+			(at 90.17 91.44 0)
+			(effects
+				(font
+					(size 1.27 1.27)
+				)
+				(hide yes)
+			)
+		)
+		(pin "1"
+		)
+		(instances
+			(project "gaia_obc"
+				(path "/049f7784-e0f9-4d41-b308-330ac61e4408/fbf62360-00e1-4059-a494-d7d297b53182"
+					(reference "#PWR0193")
+					(unit 1)
+				)

Commit message: neptune 1.3 production
Other:
- title: GAIA On-Board Computer -> Neptune On-Board Computer

Commit message: v1.4 - adding interrupt for lora
Connections:
- net LORA_DIO0: now reaches U16.14 (DIO0)
- no-connect marks 15 -> 14
Changed lines of the file:
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@@
 	(title_block
 		(title "Neptune On-Board Computer")
-		(date "2025-12-12")
-		(rev "1.3")
+		(date "2025-12-28")
+		(rev "1.4")
 	)
 	(polyline
@@
 	)
 	(no_connect
-		(at 83.82 171.45)
-	)
-	(no_connect
 		(at 45.72 109.22)
 	)
@@
 		)
 	)
+	(hierarchical_label "LORA_DIO0"
+		(shape bidirectional)
+		(at 83.82 171.45 0)
+		(effects
+			(font
+				(size 1.27 1.27)
+			)
+			(justify left)
+		)
+	)
