File: gaia_obc.kicad_sch (KiCad schematic)
At the start: 59 parts, among them J1 USB_C_Receptacle_USB2.0_16P, J2 Conn_02x10_Odd_Even, J3 Conn_02x10_Odd_Even, Q1 IRLML6244, SW1 SW_Push, SW2 SW_Push, U1 MCP23017_ML, U2 USBLC6-2P6, U3 ESP32-S3-PICO-1-N8R2

Commit message: Cleaning up schematics
Other:
- company: OnionSAT -> (none)
- title: Onboard Computer -> GAIA On-Board Computer
- moved on the sheet: D3, D4, D5, D6, D7

Commit message: v1.1-pre4 - fixing capacitors, ANT connector, optimizing routes
Parts:
- C4: footprint Capacitor_SMD:C_0402_1005Metric -> Capacitor_SMD:C_0603_1608Metric
Changed lines of the file:
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@@
 			)
 		)
-		(property "Footprint" "Capacitor_SMD:C_0402_1005Metric"
+		(property "Footprint" "Capacitor_SMD:C_0603_1608Metric"
 			(at 76.2 71.12 0)
 			(effects
