File: gaia_obc_psu.kicad_sch (KiCad schematic)
At the start: 72 parts, among them IC1 MAX17048G+T10, Q2 FS8205A, SW8 SW_Slide_DPDT, U10 TPS22917DBV, U11 AP2112K-3.3, U12 DW01A, U13 AP2112K-3.0, U14 LGS4056HDB, U4 INA3221, U5 INA3221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

Commit message: finish placing components+small fixes in schema
Parts:
- added C45, C48: 100nF, Capacitor_SMD:C_0402_1005Metric, symbol Device:C_Small
- R32, R33, R34, R35, R36, R37: footprint Resistor_SMD:R_0603_1608Metric -> Resistor_SMD:R_1206_3216Metric
Connections:
- net +3.3V: now also C45.2
- net GND: now also C45.1, C48.1

Commit message: ROUTING DONE 08. 24.
Connections:
- net +3.3V: now also C48.2
- net at R49.1: now also D10.1 (K); no longer D10.2 (A)
- net at D11.1 (K): now also R50.2; no longer U14.6 (~{STDBY})
- net at D11.2 (A): now also U14.6 (~{STDBY}); no longer R50.2
- net at U14.7 (~{CHRG}): now also D10.2 (A); no longer D10.1 (K)
Other:
- moved on the sheet: D10, D11
Changed lines of the file:
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@@
 	)
 	(junction
+		(at 64.77 38.1)
+		(diameter 0)
+		(color 0 0 0 0)
+	)
+	(junction
 		(at 87.63 64.77)
 		(diameter 0)
@@
 	(wire
 		(pts
+			(xy 64.77 38.1) (xy 69.85 38.1)
+		)
+		(stroke
+			(width 0)
+			(type default)
+		)
+	)
+	(wire
+		(pts
 			(xy 153.67 29.21) (xy 153.67 26.67)
 		)
@@
 	(wire
 		(pts
+			(xy 64.77 38.1) (xy 64.77 43.18)
+		)
+		(stroke
+			(width 0)
+			(type default)
+		)
+	)
+	(wire
+		(pts
 			(xy 115.57 148.59) (xy 127 148.59)
 		)
@@
 	(wire
 		(pts
-			(xy 69.85 38.1) (xy 66.04 38.1)
-		)
-		(stroke
-			(width 0)
-			(type default)
-		)
-	)
-	(wire
-		(pts
 			(xy 41.91 133.35) (xy 41.91 142.24)
 		)
@@
 	(wire
 		(pts
-			(xy 64.77 35.56) (xy 64.77 43.18)
+			(xy 64.77 35.56) (xy 64.77 38.1)
 		)
 		(stroke
@@
 	(symbol
 		(lib_id "Device:LED_Small")
-		(at 219.71 39.37 180)
+		(at 219.71 39.37 0)
 		(unit 1)
 		(exclude_from_sim no)
@@
 		(dnp no)
 		(property "Reference" "D11"
-			(at 219.71 44.958 0)
+			(at 219.71 43.434 0)
 			(effects
 				(font
@@
 		)
 		(property "Value" "LED_Small"
-			(at 219.964 42.672 0)
+			(at 219.71 41.402 0)
 			(effects
 				(font
@@
 	(symbol
 		(lib_id "Device:LED_Small")
-		(at 219.71 36.83 180)
+		(at 219.71 36.83 0)
 		(unit 1)
 		(exclude_from_sim no)
@@
 		)
 		(property "Value" "LED_Small"
-			(at 219.71 34.544 0)
+			(at 219.71 34.29 0)
 			(effects
 				(font

Commit message: finalizing everything + creating stencil + ORDER 08. 25.
Parts:
- Q2, U10, U12, U6, U7, U8, U9: footprint Package_TO_SOT_SMD:SOT-23-6 -> gaia_obc-footprints:SOT-23-6
- U11: footprint Package_TO_SOT_SMD:SOT-23-5 -> gaia_obc-footprints:SOT-23-6
- U13: footprint Package_TO_SOT_SMD:SOT-23-5 -> gaia_obc-footprints:SOT-23-5
- U14: footprint Package_DFN_QFN:DFN-8-1EP_3x3mm_P0.65mm_EP1.55x2.4mm -> gaia_obc-footprints:DFN-8-1EP_3x3mm_P0.65mm_EP1.55x2.4mm
- U4, U5: footprint Package_DFN_QFN:Texas_RGV0016A_VQFN-16-1EP_4x4mm_P0.65mm_EP2.1x2.1mm -> gaia_obc-footprints:Texas_RGV0016A_VQFN-16-1EP_4x4mm_P0.65mm_EP2.1x2.1mm
Changed lines of the file:
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@@
 			)
 		)
-		(property "Footprint" "Package_DFN_QFN:Texas_RGV0016A_VQFN-16-1EP_4x4mm_P0.65mm_EP2.1x2.1mm"
+		(property "Footprint" "gaia_obc-footprints:Texas_RGV0016A_VQFN-16-1EP_4x4mm_P0.65mm_EP2.1x2.1mm"
 			(at 62.23 33.02 0)
 			(effects
@@
 			)
 		)
-		(property "Footprint" "Package_TO_SOT_SMD:SOT-23-6"
+		(property "Footprint" "gaia_obc-footprints:SOT-23-6"
 			(at 137.16 138.43 0)
 			(effects
@@
 			)
 		)
-		(property "Footprint" "Package_TO_SOT_SMD:SOT-23-5"
+		(property "Footprint" "gaia_obc-footprints:SOT-23-5"
 			(at 227.33 141.605 0)
 			(effects
@@
 			)
 		)
-		(property "Footprint" "Package_TO_SOT_SMD:SOT-23-6"
+		(property "Footprint" "gaia_obc-footprints:SOT-23-6"
 			(at 137.16 46.99 0)
 			(effects
@@
 			)
 		)
-		(property "Footprint" "Package_TO_SOT_SMD:SOT-23-6"
+		(property "Footprint" "gaia_obc-footprints:SOT-23-6"
 			(at 214.63 78.74 0)
 			(effects
@@
 			)
 		)
-		(property "Footprint" "Package_DFN_QFN:Texas_RGV0016A_VQFN-16-1EP_4x4mm_P0.65mm_EP2.1x2.1mm"
+		(property "Footprint" "gaia_obc-footprints:Texas_RGV0016A_VQFN-16-1EP_4x4mm_P0.65mm_EP2.1x2.1mm"
 			(at 62.23 124.46 0)
 			(effects
@@
 			)
 		)
-		(property "Footprint" "Package_TO_SOT_SMD:SOT-23-5"
+		(property "Footprint" "gaia_obc-footprints:SOT-23-6"
 			(at 137.16 169.545 0)
 			(effects
@@
 			)
 		)
-		(property "Footprint" "Package_DFN_QFN:DFN-8-1EP_3x3mm_P0.65mm_EP1.55x2.4mm"
+		(property "Footprint" "gaia_obc-footprints:DFN-8-1EP_3x3mm_P0.65mm_EP1.55x2.4mm"
 			(at 235.458 59.69 0)
 			(effects
@@
 			)
 		)
-		(property "Footprint" "Package_TO_SOT_SMD:SOT-23-6"
+		(property "Footprint" "gaia_obc-footprints:SOT-23-6"
 			(at 222.504 90.678 0)
 			(effects
@@
 			)
 		)
-		(property "Footprint" "Package_TO_SOT_SMD:SOT-23-6"
+		(property "Footprint" "gaia_obc-footprints:SOT-23-6"
 			(at 137.16 77.47 0)
 			(effects
@@
 			)
 		)
-		(property "Footprint" "Package_TO_SOT_SMD:SOT-23-6"
+		(property "Footprint" "gaia_obc-footprints:SOT-23-6"
 			(at 137.16 107.95 0)
 			(effects
@@
 			)
 		)
-		(property "Footprint" "Package_TO_SOT_SMD:SOT-23-6"
+		(property "Footprint" "gaia_obc-footprints:SOT-23-6"
 			(at 137.16 16.51 0)
 			(effects

Commit message: Cleaning up schematics
Parts:
- D10, D11: value LED_Small -> LED
Other:
- title: (none) -> GAIA On-Board Computer

Commit message: fixing bugs v1.1-pre1
Parts:
- U11: footprint gaia_obc-footprints:SOT-23-6 -> gaia_obc-footprints:SOT-23-5
Changed lines of the file:
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@@
 			)
 		)
-		(property "Footprint" "gaia_obc-footprints:SOT-23-6"
+		(property "Footprint" "gaia_obc-footprints:SOT-23-5"
 			(at 137.16 169.545 0)
 			(effects

Commit message: v1.1-pre4 - fixing capacitors, ANT connector, optimizing routes
Parts:
- C33, C35, C37: footprint Capacitor_SMD:C_0402_1005Metric -> Capacitor_SMD:C_0603_1608Metric
Changed lines of the file:
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@@
 			)
 		)
-		(property "Footprint" "Capacitor_SMD:C_0402_1005Metric"
+		(property "Footprint" "Capacitor_SMD:C_0603_1608Metric"
 			(at 246.38 27.94 0)
 			(effects
@@
 			)
 		)
-		(property "Footprint" "Capacitor_SMD:C_0402_1005Metric"
+		(property "Footprint" "Capacitor_SMD:C_0603_1608Metric"
 			(at 227.33 24.13 0)
 			(effects
@@
 			)
 		)
-		(property "Footprint" "Capacitor_SMD:C_0402_1005Metric"
+		(property "Footprint" "Capacitor_SMD:C_0603_1608Metric"
 			(at 207.01 119.38 0)
 			(effects
