File: gaia-obc-stencil/gaia-obc-stencil.kicad_pcb (KiCad board)
At the start: 2 copper layers, 0.6 x 9 mm, 171 parts, among them IC1 MAX17048G+T10, J1 USB_C_Receptacle_USB2.0_16P, J2 Conn_02x10_Odd_Even, J3 Conn_02x10_Odd_Even, J5 Micro_SD_Card_Det2, Q1 IRLML6244, Q2 FS8205A, Q3 BSS138, SW1 SW_Push, SW2 SW_Push, SW3 SW_Push, SW4 SW_Push, SW5 SW_Push, SW6 SW_Push, SW7 SW_Push, SW8 SW_Slide_DPDT, U1 MCP23017_ML, U10 TPS22917DBV, U11 AP2112K-3.3, U12 DW01A, U13 AP2112K-3.0, U14 LGS4056HDB, U15 CD-PA1616, U16 RFM95W-868S2, U17 BME280, U2 USBLC6-2P6, U3 ESP32-S3-PICO-1-N8R2, U4 INA3221, U5 INA3221, U6 TPS22917DBV, U7 TPS22917DBV, U8 TPS22917DBV, U9 TPS22917DBV

Commit message: fixing stencil
Parts:
- AE1, C1, C10, C11, C12, C13, C14, C15, C16, C17, C18, C2, C24, C25, C26, C3, C32, C33, C34, C35, C36, C37, C38, C39, C4, C40, C42, C43, C44, C45, C46, C47, C48, C5, C6, C8, C9, IC1 (x2), J1, J2, J3, J5, L1, Q2, Q3, R1, R13, R14, R15, R16, R17, R18, R2, R20, R23, R24, R25, R26, R27, R28, R29, R3, R30, R31, R32, R33, R34, R35, R36, R37, R4, R48, R5, R51, R53, R54, R55, R59, R60, U1 (x2), U10, U11, U12, U13, U14 (x2), U16, U17 (x2), U2 (x2), U3 (x2), U4 (x2), U5 (x2), U6, U7, U8, U9: moved to F.Cu
- U18: moved to B.Cu
- moved U14 91.4 mm to (32.0, 134.2), turned to 0 degrees
- moved R1 90.1 mm to (122.8, 129.2), turned to 180 degrees
- moved R2 90.1 mm to (122.8, 128.3), turned to 180 degrees
- moved R3 90.1 mm to (122.8, 130.2), turned to 180 degrees
- moved C1 89.2 mm to (122.3, 131.6)
- moved J2 84.1 mm to (119.8, 117.3), turned to 0 degrees
- moved C2 83.0 mm to (119.2, 135.5), turned to 0 degrees
- moved IC1 81.7 mm to (36.9, 132.7), turned to 0 degrees
- moved U1 81.0 mm to (118.2, 131.4)
- moved AE1 80.7 mm to (118.1, 99.1), turned to -135 degrees
- moved U2 78.8 mm to (38.3, 135.5)
- moved C40 75.6 mm to (115.5, 136.7), turned to 180 degrees
- moved C42 75.6 mm to (115.5, 137.6), turned to 180 degrees
- moved C10 73.3 mm to (114.4, 104.3)
- moved C46 72.5 mm to (113.9, 98.9), turned to 0 degrees
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